Commit message: gazebo configurado e casa mobilhada

File: src/rm_description/urdf/differential_robot.xacro (robot description, xacro)
@@ -82,5 +82,5 @@
     mass="${wheel_1_mass}"
     material="red"/>
-  <joint name="right_wheel_joint" type="continuous">
+  <joint name="left_wheel_joint" type="continuous">
     <parent link="base_link"/>
     <child link="right_wheel"/>
@@ -98,5 +98,5 @@
     mass="${wheel_2_mass}"
     material="red"/>
-  <joint name="left_wheel_joint" type="continuous">
+  <joint name="right_wheel_joint" type="continuous">
     <parent link="base_link"/>
     <child link="left_wheel"/>

File: src/rm_description/urdf/dr_properties.xacro (robot description, xacro)
@@ -6,14 +6,14 @@
   <!-- ============================================ -->
   <!-- Propriedades do Chassis -->
-  <xacro:property name="chassis_length" value="0.3"/>
+  <xacro:property name="chassis_length" value="0.4"/>
   <xacro:property name="chassis_width" value="0.3"/>
   <xacro:property name="chassis_height" value="0.1"/>
   <xacro:property name="chassis_mass" value="2.0"/>
   <!-- Propriedades da Wheel 1 -->
-  <xacro:property name="wheel_1_length" value="0.05"/>
+  <xacro:property name="wheel_1_length" value="0.055"/>
   <xacro:property name="wheel_1_radius" value="0.08"/>
   <xacro:property name="wheel_1_mass" value="1.0"/>
   <!-- Propriedades da Wheel 2 -->
-  <xacro:property name="wheel_2_length" value="0.05"/>
+  <xacro:property name="wheel_2_length" value="0.055"/>
   <xacro:property name="wheel_2_radius" value="0.08"/>
   <xacro:property name="wheel_2_mass" value="1.0"/>

Commit message: Sensores adicionados

File: src/rm_description/urdf/differential_robot.xacro (robot description, xacro)
@@ -33,6 +33,8 @@
     $(find package_name) retorna o caminho do pacote ROS
   -->
-  <xacro:include filename="$(find rm_description)/urdf/dr_properties.xacro"/>
-  <xacro:include filename="$(find rm_description)/urdf/dr_macros.xacro"/>
+  <xacro:include filename="$(find rm_description)/urdf/properties.xacro"/>
+  <xacro:include filename="$(find rm_description)/urdf/wheels.xacro"/>
+  <xacro:include filename="$(find rm_description)/urdf/gazebo_control.xacro" />
+  <xacro:include filename="$(find rm_description)/urdf/sensors.xacro" />
   <!-- ==================== -->
   <!-- BASE FOOTPRINT       -->
@@ -44,12 +46,12 @@
   <link name="base_link">
     <visual>
-      <origin xyz="0 0 0" rpy="0 0 0"/>
+      <origin xyz="${offset} 0 0" rpy="0 0 0"/>
       <geometry>
         <box size="${chassis_length} ${chassis_width} ${chassis_height}"/>
       </geometry>
-      <material name="black"/>
+      <material name="dark_gray"/>
     </visual>
     <collision>
-      <origin xyz="0 0 0" rpy="0 0 0"/>
+      <origin xyz="${offset} 0 0" rpy="0 0 0"/>
       <geometry>
         <box size="${chassis_length} ${chassis_width} ${chassis_height}"/>
@@ -57,5 +59,5 @@
     </collision>
     <inertial>
-      <origin xyz="0 0 0" rpy="0 0 0"/>
+      <origin xyz="${offset} 0 0" rpy="0 0 0"/>
       <mass value="${chassis_mass}"/>
       <inertia
@@ -70,5 +72,5 @@
     <parent link="base_footprint"/>
     <child link="base_link"/>
-    <origin xyz="0 0 ${wheel_1_radius}" rpy="0 0 0"/>
+    <origin xyz="0 0 ${wheel_radius}" rpy="0 0 0"/>
   </joint>
   <!-- ==================== -->
@@ -78,12 +80,12 @@
   <xacro:cylinder_link_right
     name="right_wheel"
-    length="${wheel_1_length}"
-    radius="${wheel_1_radius}"
-    mass="${wheel_1_mass}"
+    length="${wheel_length}"
+    radius="${wheel_radius}"
+    mass="${wheel_mass}"
     material="red"/>
   <joint name="left_wheel_joint" type="continuous">
     <parent link="base_link"/>
     <child link="right_wheel"/>
-    <origin xyz="0 ${chassis_width/2} 0" rpy="0 0 0"/>
+    <origin xyz="0 ${chassis_width/2 + wheel_length/2} 0" rpy="0 0 0"/>
     <axis xyz="0 1 0"/>
   </joint>
@@ -94,12 +96,12 @@
   <xacro:cylinder_link_left
     name="left_wheel"
-    length="${wheel_2_length}"
-    radius="${wheel_2_radius}"
-    mass="${wheel_2_mass}"
+    length="${wheel_length}"
+    radius="${wheel_radius}"
+    mass="${wheel_mass}"
     material="red"/>
   <joint name="right_wheel_joint" type="continuous">
     <parent link="base_link"/>
     <child link="left_wheel"/>
-    <origin xyz="0 ${-chassis_width/2} 0" rpy="0 0 0"/>
+    <origin xyz="0 ${-chassis_width/2 - wheel_length/2} 0" rpy="0 0 0"/>
     <axis xyz="0 1 0"/>
   </joint>
@@ -112,9 +114,89 @@
     radius="${cw_radius}"
     mass="${cw_mass}"
-    material="gray"/>
+    material="silver"/>
   <joint name="caster_joint" type="fixed">
     <parent link="base_link"/>
     <child link="caster_ball"/>
-    <origin xyz="${chassis_length/2 - cw_radius} 0 ${-(chassis_height/2)}" rpy="0 0 0"/>
+    <origin xyz="${chassis_length/2 - cw_radius + offset} 0 ${-(chassis_height/2)}" rpy="0 0 0"/>
+  </joint>
+  <!-- ==================== -->
+  <!-- CÂMERA               -->
+  <!-- ==================== -->
+  <link name="camera">
+    <visual>
+      <!-- Desloca para que a BASE do cilindro fique na origem -->
+      <origin xyz="${-camera_length/2} 0 0" rpy="0 1.57079 0"/>
+      <geometry>
+        <cylinder radius="${camera_radius}" length="${camera_length}"/>
+      </geometry>
+      <material name="gray"/>
+    </visual>
+    <collision>
+      <origin xyz="${-camera_length/2} 0 0" rpy="0 1.57079 0"/>
+      <geometry>
+        <cylinder radius="${camera_radius}" length="${camera_length}"/>
+      </geometry>
+    </collision>
+    <inertial>
+      <origin xyz="${-camera_length/2} 0 0" rpy="0 1.57079 0"/>
+      <mass value="${camera_mass}"/>
+      <!-- Fórmula de inércia para cilindro sólido -->
+      <inertia
+        ixx="${(1/12) * camera_mass * (3*camera_radius*camera_radius + camera_length*camera_length)}"
+        ixy="0.0" ixz="0.0"
+        iyy="${(1/12) * camera_mass * (3*camera_radius*camera_radius + camera_length*camera_length)}"
+        iyz="0.0"
+        izz="${(1/2) * camera_mass * camera_radius * camera_radius}"/>
+    </inertial>
+  </link>
+  <joint name="camera_joint" type="fixed">
+  <parent link="base_link"/>
+  <child link="camera"/>
+  <origin xyz="${chassis_length/2 + offset} 0 ${chassis_height/2 + camera_radius}" rpy="0 0 0"/>
+  </joint>
+  <!-- ==================== -->
+  <!-- LIDAR               -->
+  <!-- ==================== -->
+  <link name="lidar">
+    <visual>
+      <!-- Desloca para que a BASE do cilindro fique na origem -->
+      <origin xyz="0 0 0" rpy="0 0 0"/>
+      <geometry>
+        <cylinder radius="${lidar_radius}" length="${lidar_length}"/>
+      </geometry>
+      <material name="gray"/>
+    </visual>
+    <collision>
+      <origin xyz="0 0 0" rpy="0 0 0"/>
+      <geometry>
+        <cylinder radius="${lidar_radius}" length="${lidar_length}"/>
+      </geometry>
+    </collision>
+    <inertial>
+      <origin xyz="0 0 0" rpy="0 0 0"/>
+      <mass value="${lidar_mass}"/>
+      <!-- Fórmula de inércia para cilindro sólido -->
+      <inertia
+        ixx="${(1/12) * lidar_mass * (3*lidar_radius*lidar_radius + lidar_length*lidar_length)}"
+        ixy="0.0" ixz="0.0"
+        iyy="${(1/12) * lidar_mass * (3*lidar_radius*lidar_radius + lidar_length*lidar_length)}"
+        iyz="0.0"
+        izz="${(1/2) * lidar_mass * lidar_radius * lidar_radius}"/>
+    </inertial>
+  </link>
+  <joint name="lidar_joint" type="fixed">
+  <parent link="base_link"/>
+  <child link="lidar"/>
+  <origin xyz="0 0 ${chassis_height/2 + lidar_length/2}" rpy="0 0 0"/>
+  </joint>
+  <!-- ==================== -->
+  <!-- IMU                  -->
+  <!-- ==================== -->
+  <link name="imu">
+  </link>
+  <joint name="imu_joint" type="fixed">
+  <parent link="base_link"/>
+  <child link="imu"/>
+  <origin xyz="0 0 0" rpy="0 0 0"/>
   </joint>
 </robot>

File: src/rm_description/urdf/properties.xacro (robot description, xacro)
@@ -5,34 +5,43 @@
   <!-- Contém todas as constantes e dimensões       -->
   <!-- ============================================ -->
-  <!-- Propriedades da Base -->
-  <xacro:property name="base_radius" value="0.1"/>
-  <xacro:property name="base_height" value="0.05"/>
-  <xacro:property name="base_mass" value="2.0"/>
-  <!-- TAREFA: Defina as propriedades do Link 1 -->
-  <!-- Use os valores da tabela de referência (seção 2.2) -->
-  <xacro:property name="link1_length" value="0.3"/>
-  <xacro:property name="link1_radius" value="0.03"/>
-  <xacro:property name="link1_mass" value="1.0"/>
-  <!-- TAREFA: Defina as propriedades do Link 2 -->
-  <xacro:property name="link2_length" value="0.25"/>
-  <xacro:property name="link2_radius" value="0.025"/>
-  <xacro:property name="link2_mass" value="0.8"/>
-  <!-- Propriedades do End Effector -->
-  <xacro:property name="ee_radius" value="0.02"/>
-  <xacro:property name="ee_mass" value="0.1"/>
+  <!-- Propriedades do Chassis -->
+  <xacro:property name="chassis_length" value="0.4"/>
+  <xacro:property name="chassis_width" value="0.3"/>
+  <xacro:property name="chassis_height" value="0.1"/>
+  <xacro:property name="chassis_mass" value="2.0"/>
+  <!-- Propriedades das Rodas -->
+  <xacro:property name="wheel_length" value="0.055"/>
+  <xacro:property name="wheel_radius" value="0.08"/>
+  <xacro:property name="wheel_mass" value="1.0"/>
+  <!-- Offset Rodas-->
+  <xacro:property name="offset" value="0.1"/>
+  <!-- Propriedades da Caster Wheel -->
+  <xacro:property name="cw_radius" value="0.03"/>
+  <xacro:property name="cw_mass" value="0.1"/>
+  <!-- Propriedades da Camera -->
+  <xacro:property name="camera_length" value="0.1"/>
+  <xacro:property name="camera_radius" value="0.03"/>
+  <xacro:property name="camera_mass" value="0.05"/>
+  <!-- Propriedades do lidar -->
+  <xacro:property name="lidar_length" value="0.05"/>
+  <xacro:property name="lidar_radius" value="0.05"/>
+  <xacro:property name="lidar_mass" value="0.1"/>
   <!-- ============================================ -->
   <!-- MATERIAIS (cores)                            -->
   <!-- ============================================ -->
-  <material name="gray">
+  <material name="silver">
     <color rgba="0.5 0.5 0.5 1"/>
   </material>
-  <material name="blue">
-    <color rgba="0 0 0.8 1"/>
+  <material name="gray">
+    <color rgba="0.1 0.1 0.1 1"/>
+  </material>
+  <material name="dark_gray">
+    <color rgba="0.02 0.02 0.02 1"/>
   </material>
   <material name="red">
-    <color rgba="0.8 0 0 1"/>
+    <color rgba="0.5 0 0 1"/>
   </material>
-  <material name="green">
-    <color rgba="0 0.8 0 1"/>
+  <material name="blue">
+    <color rgba="0 0 0.5 1"/>
   </material>
 </robot>

File: src/rm_description/urdf/wheels.xacro (robot description, xacro)
@@ -5,7 +5,7 @@
   <!-- Contém componentes reutilizáveis             -->
   <!-- ============================================ -->
-  <!-- ==================== -->
-  <!-- MACRO: LINK CILÍNDRICO -->
-  <!-- ==================== -->
+  <!-- ========================= -->
+  <!-- MACRO: LINK CILÍNDRICO Y+ -->
+  <!-- ========================= -->
   <!--
     Cria um link cilíndrico completo com visual, collision e inertial.
@@ -13,14 +13,14 @@
     Parâmetros:
       - name: nome do link
-      - length: comprimento do cilindro (eixo Z)
+      - length: comprimento do cilindro (eixo Y)
       - radius: raio do cilindro
       - mass: massa em kg
       - material: nome do material (definido em properties.xacro)
   -->
-  <xacro:macro name="cylinder_link" params="name length radius mass material">
+  <xacro:macro name="cylinder_link_right" params="name length radius mass material">
     <link name="${name}">
       <visual>
         <!-- Desloca para que a BASE do cilindro fique na origem -->
-        <origin xyz="0 0 ${length/2}" rpy="0 0 0"/>
+        <origin xyz="0 0 0" rpy="1.5708 0 0"/>
         <geometry>
           <cylinder radius="${radius}" length="${length}"/>
@@ -29,5 +29,5 @@
       </visual>
       <collision>
-        <origin xyz="0 0 ${length/2}" rpy="0 0 0"/>
+        <origin xyz="0 0 0" rpy="1.5708 0 0"/>
         <geometry>
           <cylinder radius="${radius}" length="${length}"/>
@@ -35,5 +35,47 @@
       </collision>
       <inertial>
-        <origin xyz="0 0 ${length/2}" rpy="0 0 0"/>
+        <origin xyz="0 0 0" rpy="1.5708 0 0"/>
+        <mass value="${mass}"/>
+        <!-- Fórmula de inércia para cilindro sólido -->
+        <inertia
+          ixx="${(1/12) * mass * (3*radius*radius + length*length)}"
+          ixy="0.0" ixz="0.0"
+          iyy="${(1/12) * mass * (3*radius*radius + length*length)}"
+          iyz="0.0"
+          izz="${(1/2) * mass * radius * radius}"/>
+      </inertial>
+    </link>
+  </xacro:macro>
+  <!-- ========================= -->
+  <!-- MACRO: LINK CILÍNDRICO Y- -->
+  <!-- ========================= -->
+  <!--
+    Cria um link cilíndrico completo com visual, collision e inertial.
+    O cilindro é posicionado com a BASE na origem do link.
+    Parâmetros:
+      - name: nome do link
+      - length: comprimento do cilindro (eixo Y)
+      - radius: raio do cilindro
+      - mass: massa em kg
+      - material: nome do material (definido em properties.xacro)
+  -->
+  <xacro:macro name="cylinder_link_left" params="name length radius mass material">
+    <link name="${name}">
+      <visual>
+        <!-- Desloca para que a BASE do cilindro fique na origem -->
+        <origin xyz="0 0 0" rpy="1.5708 0 0"/>
+        <geometry>
+          <cylinder radius="${radius}" length="${length}"/>
+        </geometry>
+        <material name="${material}"/>
+      </visual>
+      <collision>
+        <origin xyz="0 0 0" rpy="1.5708 0 0"/>
+        <geometry>
+          <cylinder radius="${radius}" length="${length}"/>
+        </geometry>
+      </collision>
+      <inertial>
+        <origin xyz="0 0 0" rpy="1.5708 0 0"/>
         <mass value="${mass}"/>
         <!-- Fórmula de inércia para cilindro sólido -->

Commit message: APS Completa

File: src/rm_description/urdf/differential_robot.xacro (robot description, xacro)
@@ -75,9 +75,25 @@
   </joint>
   <!-- ==================== -->
-  <!-- RIGHT WHEEL (Y+)      -->
+  <!-- RIGHT WHEEL      -->
   <!-- ==================== -->
   <!-- Usa cylinder_link com Y+ para posicionar o cilindro na direção positiva do eixo Y -->
-  <xacro:cylinder_link_right
+  <xacro:cylinder_link
     name="right_wheel"
+    length="${wheel_length}"
+    radius="${wheel_radius}"
+    mass="${wheel_mass}"
+    material="red"/>
+  <joint name="right_wheel_joint" type="continuous">
+    <parent link="base_link"/>
+    <child link="right_wheel"/>
+    <origin xyz="0 ${-chassis_width/2 - wheel_length/2} 0" rpy="0 0 0"/>
+    <axis xyz="0 1 0"/>
+  </joint>
+  <!-- ==================== -->
+  <!-- LEFT WHEEL      -->
+  <!-- ==================== -->
+  <!-- Usa cylinder_link com Y- para posicionar o cilindro na direção negativa do eixo Y -->
+  <xacro:cylinder_link
+    name="left_wheel"
     length="${wheel_length}"
     radius="${wheel_radius}"
@@ -86,22 +102,6 @@
   <joint name="left_wheel_joint" type="continuous">
     <parent link="base_link"/>
-    <child link="right_wheel"/>
+    <child link="left_wheel"/>
     <origin xyz="0 ${chassis_width/2 + wheel_length/2} 0" rpy="0 0 0"/>
-    <axis xyz="0 1 0"/>
-  </joint>
-  <!-- ==================== -->
-  <!-- LEFT WHEEL (Y-)      -->
-  <!-- ==================== -->
-  <!-- Usa cylinder_link com Y- para posicionar o cilindro na direção negativa do eixo Y -->
-  <xacro:cylinder_link_left
-    name="left_wheel"
-    length="${wheel_length}"
-    radius="${wheel_radius}"
-    mass="${wheel_mass}"
-    material="red"/>
-  <joint name="right_wheel_joint" type="continuous">
-    <parent link="base_link"/>
-    <child link="left_wheel"/>
-    <origin xyz="0 ${-chassis_width/2 - wheel_length/2} 0" rpy="0 0 0"/>
     <axis xyz="0 1 0"/>
   </joint>
@@ -153,5 +153,5 @@
   <parent link="base_link"/>
   <child link="camera"/>
-  <origin xyz="${chassis_length/2 + offset} 0 ${chassis_height/2 + camera_radius}" rpy="0 0 0"/>
+  <origin xyz="${chassis_length/2 + offset + camera_length/2} 0 0" rpy="0 0 0"/>
   </joint>
   <!-- ==================== -->

File: src/rm_description/urdf/properties.xacro (robot description, xacro)
@@ -20,10 +20,10 @@
   <xacro:property name="cw_mass" value="0.1"/>
   <!-- Propriedades da Camera -->
-  <xacro:property name="camera_length" value="0.1"/>
+  <xacro:property name="camera_length" value="0.05"/>
   <xacro:property name="camera_radius" value="0.03"/>
   <xacro:property name="camera_mass" value="0.05"/>
   <!-- Propriedades do lidar -->
-  <xacro:property name="lidar_length" value="0.05"/>
-  <xacro:property name="lidar_radius" value="0.05"/>
+  <xacro:property name="lidar_length" value="0.08"/>
+  <xacro:property name="lidar_radius" value="0.06"/>
   <xacro:property name="lidar_mass" value="0.1"/>
   <!-- ============================================ -->

File: src/rm_description/urdf/sensors.xacro (robot description, xacro)
@@ -33,8 +33,8 @@
                 <scan>
                     <horizontal>
-                        <samples>360</samples>
+                        <samples>720</samples>
                         <resolution>1</resolution>
-                        <min_angle>-3.14</min_angle>
-                        <max_angle>3.14</max_angle>
+                        <min_angle>-3.1415</min_angle>
+                        <max_angle>3.1415</max_angle>
                     </horizontal>
                 </scan>

File: src/rm_description/urdf/wheels.xacro (robot description, xacro)
@@ -6,5 +6,5 @@
   <!-- ============================================ -->
   <!-- ========================= -->
-  <!-- MACRO: LINK CILÍNDRICO Y+ -->
+  <!-- MACRO: LINK CILÍNDRICO  -->
   <!-- ========================= -->
   <!--
@@ -18,47 +18,5 @@
       - material: nome do material (definido em properties.xacro)
   -->
-  <xacro:macro name="cylinder_link_right" params="name length radius mass material">
-    <link name="${name}">
-      <visual>
-        <!-- Desloca para que a BASE do cilindro fique na origem -->
-        <origin xyz="0 0 0" rpy="1.5708 0 0"/>
-        <geometry>
-          <cylinder radius="${radius}" length="${length}"/>
-        </geometry>
-        <material name="${material}"/>
-      </visual>
-      <collision>
-        <origin xyz="0 0 0" rpy="1.5708 0 0"/>
-        <geometry>
-          <cylinder radius="${radius}" length="${length}"/>
-        </geometry>
-      </collision>
-      <inertial>
-        <origin xyz="0 0 0" rpy="1.5708 0 0"/>
-        <mass value="${mass}"/>
-        <!-- Fórmula de inércia para cilindro sólido -->
-        <inertia
-          ixx="${(1/12) * mass * (3*radius*radius + length*length)}"
-          ixy="0.0" ixz="0.0"
-          iyy="${(1/12) * mass * (3*radius*radius + length*length)}"
-          iyz="0.0"
-          izz="${(1/2) * mass * radius * radius}"/>
-      </inertial>
-    </link>
-  </xacro:macro>
-  <!-- ========================= -->
-  <!-- MACRO: LINK CILÍNDRICO Y- -->
-  <!-- ========================= -->
-  <!--
-    Cria um link cilíndrico completo com visual, collision e inertial.
-    O cilindro é posicionado com a BASE na origem do link.
-    Parâmetros:
-      - name: nome do link
-      - length: comprimento do cilindro (eixo Y)
-      - radius: raio do cilindro
-      - mass: massa em kg
-      - material: nome do material (definido em properties.xacro)
-  -->
-  <xacro:macro name="cylinder_link_left" params="name length radius mass material">
+  <xacro:macro name="cylinder_link" params="name length radius mass material">
     <link name="${name}">
       <visual>
